Commit message: 手写控制器实验成功。

File: gazebo_pkg/urdf/waking_robot.xacro (robot description, xacro)
@@ -8,8 +8,8 @@
                <inertial>
                        <mass value="${mass}" />
-                       <inertia ixx="0.1" ixy="0.0"
+                       <inertia ixx="0.01" ixy="0.0"
                                 ixz="0.0"
-                                iyy="0.1" iyz="0.0"
-                                izz="0.1" />
+                                iyy="0.01" iyz="0.0"
+                                izz="0.01" />
                </inertial>
 	</xacro:macro>
@@ -271,10 +271,11 @@
  </gazebo>
   <!-- ros_control plugin -->
-<!--   <gazebo>
+  <!-- 取消了注释 -->
+ <gazebo>
     <plugin name="gazebo_ros_control" filename="libgazebo_ros_control.so">
       <robotNamespace>/robot</robotNamespace>
        <legacyModeNS> true </legacyModeNS>
     </plugin>
-  </gazebo> -->
+  </gazebo>
   <!-- camera_link -->
   <gazebo reference="camera_link">
@@ -373,9 +374,12 @@
     <wheelSeparation>0.26</wheelSeparation>
     <wheelDiameter>0.12</wheelDiameter>
+    <covariance_x>0.000100</covariance_x>
+    <covariance_y>0.000100</covariance_y>
+    <covariance_yaw>0.010000</covariance_yaw>
     <torque>2</torque>
-    <commandTopic>vel_ctrl</commandTopic> <!--使用cmd_vel话题作为速度命令接收-->
+    <commandTopic>cmd_vel</commandTopic>
     <odometryTopic>odom</odometryTopic>
     <odometryFrame>odom</odometryFrame>
-    <robotBaseFrame>dummy</robotBaseFrame>
+    <robotBaseFrame>dummy</robotBaseFrame> <!--default base_footprint-->
     <broadcastTF>1</broadcastTF>
   </plugin>
